File: HW/pcb/drone_controller.brd (EAGLE design)
At the start: 43.5 x 83.8 mm, 20 parts, among them J1 SM08B-SRSS-TB, U1 ICM-20600, U2 VXO7805-500

Commit message: ordered V1.1 of drone PCB
Parts:
- removed A1: 113990105, 113990105:SEEED_113990105
- added C10: 0.1uF, capacitor-wima:C2.5-3
- added C11: 1uF, capacitor-wima:C2.5-3
- added C3, C8: 0.1uF, rcl:C0603
- added C9: 10uF, capacitor-wima:C2.5-3
- added J2: 629105136821, Eagle_WR-USB (rev22c):629105136821
- added JP1: (no value), pinhead:1X05
- added R4, R5: 0R, rcl:0204/7
- added R9: 10K, rcl:0204/7
- added SJ1, SJ2, SJ3: (no value), jumper:SJ
- added SV3: (no value), con-lstb:MA04-1
- added U3: M24C02-WMN6TP, M24C02-WMN6TP:SOIC127P600X175-8N
- added U4: ESP32-C3-MINI-1-N4, ESP32-C3-MINI-1-N4:XCVR_ESP32-C3-MINI-1-N4
- U2: value VXO7805-500 -> PXO7803-500-S; device VXO7805-500:CONV_VXO7805-500 -> PXO7803-500-S:CONV_PXO7803-500-S
- moved R3 31.2 mm to (6.99, 62.9)
- moved R7 31.2 mm to (6.99, 65.4), turned to 180 degrees
- moved U1 10.2 mm to (23.1, 36.8)
- moved SV2 9.53 mm to (16.5, 37.5)
- moved C1 8.91 mm to (11.4, 25.4), turned to 0 degrees
- moved C2 8.89 mm to (5.71, 25.4), turned to 0 degrees
- moved C5 8.47 mm to (27.9, 23.5)
- moved C6 8.35 mm to (22.9, 23.5)
- moved SV1 5.81 mm to (23.1, 14.6)
- moved U2 5.75 mm to (10.8, 28.6), turned to 180 degrees
- moved C4 2.54 mm to (33.0, 22.9)
- moved C7 1.27 mm to (33.0, 27.9)
- moved J1 0.63 mm to (3.30, 56.5), flipped to the bottom, turned to 90 degrees
- moved R1 0.63 mm to (38.7, 34.3)
- moved R2 0.63 mm to (38.7, 36.8)
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Connections:
- removed net 5V: A1.J1_15, C2.1, U2.3
- removed net INT: SV2.1
- removed net N$17: SV2.4
- removed net N$18: SV2.3
- removed net N$19: SV2.2
- new net N$2: JP1.5
- new net N$3: C11.1, R9.1, U4.8
- new net N$6: SJ1.2, U3.1
- new net N$7: SJ2.2, U3.2
- new net N$8: SJ3.2, U3.3
- new net RX: SV3.3, U4.30
- new net TX: SV3.2, U4.31
- new net USB_D_N: C3.1, J2.2, R4.2
- new net USB_D_P: C8.1, J2.3, R5.2
- new net USB_RD_N: R4.1, U4.26
- new net USB_RD_P: R5.1, U4.27
- new net USB_VCC: J2.1
- net 3V3: now also C10.1, C2.1, C9.1, R9.2, SJ1.1, SJ2.1, SJ3.1, SV3.1, U2.3, U3.8, U4.3; no longer A1.J1_11, A1.J2_15, A1.J2_6
- net GND: now also C10.2, C11.2, C3.2, C8.2, C9.2, J2.5, JP1.1, SV3.4, U3.4, U3.7, U4.1, U4.11, U4.14, U4.2, U4.36, U4.37, U4.38, U4.39, U4.40, U4.41, U4.42, U4.43, U4.44, U4.45, U4.46, U4.47, U4.48, U4.49_1, U4.49_2, U4.49_3, U4.49_4, U4.49_5, U4.49_6, U4.49_7, U4.49_8, U4.49_9, U4.50, U4.51, U4.52, U4.53; no longer A1.J1_10, A1.J1_14, A1.J2_14, A1.J2_7
- net GPIO_BATT_SOC: now also U4.12; no longer A1.J1_1
- net GPIO_LED_HEARTBEAT: now also U4.20; no longer A1.J2_4
- net GPIO_LED_WIFI_CONN: now also U4.23; no longer A1.J2_10
- net GPIO_LED_WIFI_RX: now also U4.19; no longer A1.J2_5
- net PWM_MOTOR_FL: now also JP1.3, U4.13; no longer A1.J2_8
- net PWM_MOTOR_FR: now also JP1.2, U4.5; no longer A1.J2_9
- net PWM_MOTOR_RL: now also U4.6; no longer A1.J2_11
- net PWM_MOTOR_RR: now also JP1.4, U4.18; no longer A1.J2_1
- net SCL: now also U3.6, U4.22; no longer A1.J2_2
- net SDA: now also U3.5, U4.21; no longer A1.J2_3
Routing:
- net SDA: track 167.9 -> 68.3 mm, vias 2 -> 0
- net GND: track 0.00 -> 59.2 mm, vias 42 -> 2
- net 5V: track 54.2 -> 0.00 mm, vias 2 -> 0
- net 3V3: track 138.7 -> 183.4 mm, vias 0 -> 4
- net PWM_MOTOR_RR: track 84.2 -> 42.7 mm, vias 2 -> 1
- net GPIO_BATT_SOC: track 61.3 -> 20.7 mm
- net PWM_MOTOR_RL: track 47.9 -> 11.2 mm, vias 0 -> 1
- net SCL: track 120.3 -> 85.7 mm
- net PWM_MOTOR_FL: track 66.3 -> 39.6 mm
- net TX: track 0.00 -> 25.2 mm, vias 0 -> 2
- net N$3: track 0.00 -> 21.2 mm, vias 0 -> 1
- net USB_D_P: track 0.00 -> 20.9 mm
- net RX: track 0.00 -> 20.3 mm
- net AD0: track 49.3 -> 29.2 mm, vias 4 -> 1
- net USB_D_N: track 0.00 -> 18.0 mm
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Other:
- board size 43.5 x 83.8 mm -> 43.5 x 70.5 mm
- board text added: "BLHeli: 1 2 3 4 GND"
- board text added: "Drone v1.1"
- board text added: "IMU Offset from (X,Y): (0,4.76) mm"
- board text added: "LiPO SOC Cal"
- board text added: "Mem Addr Set"
- board text added: "Serial: GND RX TX VCC"
- board text removed: "Drone v1.0"
- board text removed: "FLM"
- board text removed: "FRM"
- board text removed: "IMU Offset from (X,Y): (0,17.78) mm"
- board text removed: "RLM"
- board text removed: "RRM"
